Commit message: urdf modifications

File: urdf/arm.urdf.xacro (robot description, xacro)
@@ -1,4 +1,5 @@
 <?xml version="1.0"?>
-<robot name="arm">
+<robot name="arm" xmlns:xacro="http://ros.org/wiki/xacro">
+	<xacro:include filename="$(find hector_sensors_description)/urdf/asus_camera.urdf.xacro" />
 	<link name="base_link">
 		<visual>
@@ -45,4 +46,14 @@
 		</visual>
 	</link>
+	<xacro:asus_camera name="camera" parent="base_link">
+		<origin xyz="0.195 0.0 0.165" rpy="0 0 0"/>
+	</xacro:asus_camera>
+	<link name="scan">
+	</link>
+	<joint name="scan_joint" type="fixed">
+		<parent link="camera_depth_frame"/>
+		<child link="scan"/>
+		<origin xyz="0.0 0.0 0.0" rpy="0 0 0"/>
+	</joint>
 	<joint name="front_wheel_joint" type="fixed">
 		<parent link="base_link"/>

Commit message: urdf cleanup

File: urdf/arm.urdf.xacro (robot description, xacro)
@@ -49,11 +49,4 @@
 		<origin xyz="0.195 0.0 0.165" rpy="0 0 0"/>
 	</xacro:asus_camera>
-	<link name="scan">
-	</link>
-	<joint name="scan_joint" type="fixed">
-		<parent link="camera_depth_frame"/>
-		<child link="scan"/>
-		<origin xyz="0.0 0.0 0.0" rpy="0 0 0"/>
-	</joint>
 	<joint name="front_wheel_joint" type="fixed">
 		<parent link="base_link"/>
