Commit message: added move_base, configs, edited urdf

File: urdf/arm.urdf (robot description, URDF)
Before this commit: robot arm, 13 links, 12 joints
Links:
- removed link antenna
- removed link front_left_eye
- removed link front_left_wheel
- removed link front_lower_left_eye
- removed link front_lower_right_eye
- removed link front_right_eye
- removed link front_right_wheel
- removed link platform
- removed link scan
- removed link sonar_forward_lower
- added link front_wheel; visual cylinder length=0.002 radius=0.025
- link aft_left_wheel: geometry visual cylinder length=0.002 radius=0.025
- link aft_right_wheel: geometry visual cylinder length=0.002 radius=0.025
- link base_link: geometry visual box size=0.30 0.22 0.015
Joints:
- removed joint antenna_joint
- removed joint front_left_eye_joint
- removed joint front_left_wheel_joint
- removed joint front_lower_left_eye_joint
- removed joint front_lower_right_eye_joint
- removed joint front_right_eye_joint
- removed joint front_right_wheel_joint
- removed joint platform_joint
- removed joint scan_joint
- removed joint sonar_forward_lower_join
- added joint front_wheel_joint: type fixed, parent base_link, child front_wheel, origin xyz=0.17 0.0 0.025 rpy=0 0 0
- joint aft_left_wheel_joint: origin xyz=-0.08 0.05 0.03 rpy=0 0 0 -> xyz=0.0 0.05 0.025 rpy=0 0 0
- joint aft_right_wheel_joint: origin xyz=-0.08 -0.05 0.03 rpy=0 0 0 -> xyz=0.0 -0.05 0.025 rpy=0 0 0

Commit message: publish joint messages, added gripper 35978

File: urdf/arm.urdf (robot description, URDF)
Before this commit: robot wild_thumper, 8 links, 7 joints
Links:
- link gripper_pole1: geometry visual cylinder length=0.03 radius=0.045
- link gripper_pole2: geometry visual cylinder length=0.015 radius=0.03
- link left_gripper: geometry visual mesh filename=package://arm_ros_conn/meshes/35978.stl scale=0.001 0.001 0.001
- link right_gripper: geometry visual mesh filename=package://arm_ros_conn/meshes/35978.stl scale=0.001 0.001 0.001
Joints:
- joint gripper_joint_2: origin xyz=0.055 0.0 0.0 rpy=0 0 0 -> xyz=0.06 0.0 0.0 rpy=0 0 0
- joint left_gripper_joint: limit lower=0.0 upper=0.548 effort=1000.0 velocity=1.0 -> lower=0.0 upper=0.35 effort=1000.0 velocity=1.0; origin xyz=0 0.01 0 rpy=0 0 0 -> xyz=0.02 0.01 0 rpy=0 0 0
- joint right_gripper_joint: limit lower=0.0 upper=0.548 effort=1000.0 velocity=1.0 -> lower=0.0 upper=0.35 effort=1000.0 velocity=1.0; origin xyz=0 -0.01 0 rpy=0 0 0 -> xyz=0.02 -0.01 0 rpy=0 0 0

Commit message: arm_ros_conn: allow to preempt

File: urdf/arm.urdf (robot description, URDF)
Before this commit: robot arm, 8 links, 7 joints
Joints:
- joint base_to_link1: limit lower=0.0 upper=5.672320068981571 effort=1000.0 velocity=1.0 -> lower=-5.672320068981571 upper=0.0 effort=1000.0 velocity=1.0
- joint gripper_joint_1: limit lower=-0.6981317007977319 upper=7.679448708775051 effort=1000.0 velocity=1.0 -> lower=-7.679448708775051 upper=0.6981317007977319 effort=1000.0 velocity=1.0
- joint link_2_3_joint: limit lower=0.0 upper=3.141592653589793 effort=1000.0 velocity=1.0 -> lower=-3.141592653589793 upper=0.0 effort=1000.0 velocity=1.0

Commit message: added meshes

File: urdf/arm.urdf (robot description, URDF)
Before this commit: robot arm, 8 links, 7 joints
Links:
- removed link gripper_pole1
- removed link gripper_pole2
- added link gripper_pole
- added link link4; visual cylinder length=0.03 radius=0.045
- added link link5; visual mesh filename=package://arm_ros_conn/meshes/31019.stl scale=1 1 1
- link base_link: geometry visual mesh filename=package://arm_ros_conn/meshes/32985.stl scale=1 1 1
- link link1: geometry visual box size=0.06 0.03 0.123
Joints:
- removed joint gripper_joint_1
- removed joint gripper_joint_2
- added joint gripper_pole_joint: type fixed, parent link5, child gripper_pole
- added joint link_3_4_joint: type continuous, parent link3, child link4, origin xyz=0 0.135 0.0 rpy=1.57075 0 1.57075, axis 1 0 0, limit lower=-7.679448708775051 upper=0.6981317007977319 effort=1000.0 velocity=1.0
- added joint link_4_5_joint: type continuous, parent link4, child link5, origin xyz=0.06 0.0 0.0 rpy=0 0 0, axis 0 1 0, limit lower=-1.5707963267948966 upper=1.5707963267948966 effort=1000.0 velocity=1.0
- joint base_to_link1: origin (none) -> xyz=0 0.099 0
- joint left_gripper_joint: parent gripper_pole2 -> gripper_pole
- joint right_gripper_joint: parent gripper_pole2 -> gripper_pole

Commit message: urdf fixes

File: urdf/arm.urdf (robot description, URDF)
Before this commit: robot arm, 9 links, 8 joints
Links:
- added link arm_base; visual mesh filename=package://arm_ros_conn/meshes/32985.stl
- link base_link: geometry 
- link link5: geometry visual mesh filename=package://arm_ros_conn/meshes/31019.stl
Joints:
- removed joint base_to_link1
- added joint arm_base_to_link1: type continuous, parent arm_base, child link1, origin xyz=0 0.099 0, axis 0 0 1, limit lower=-5.672320068981571 upper=0.0 effort=1000.0 velocity=1.0
- added joint base_link_to_arm_base: type fixed, parent base_link, child arm_base, origin xyz=0 0 0.00375
- joint link_1_2_joint: origin xyz=0.0 0.0 0.135 rpy=1.57075 0 0 -> xyz=0.0 0.0 0.123 rpy=1.57075 0 0

Commit message: use revolut instead of continous joints

File: urdf/arm.urdf (robot description, URDF)
Before this commit: robot arm, 10 links, 9 joints
Joints:
- joint arm_base_to_link1: type continuous -> revolute
- joint link_1_2_joint: type continuous -> revolute
- joint link_2_3_joint: type continuous -> revolute
- joint link_3_4_joint: limit lower=-7.679448708775051 upper=0.6981317007977319 effort=1000.0 velocity=1.0 -> lower=-5.4978 upper=-0.15708 effort=1000.0 velocity=1.0; type continuous -> revolute
- joint link_4_5_joint: type continuous -> revolute

Commit message: fixes for new urdf

File: urdf/arm.urdf (robot description, URDF)
Before this commit: robot arm, 10 links, 9 joints
Joints:
- joint link_3_4_joint: limit lower=-5.4978 upper=-0.15708 effort=1000.0 velocity=1.0 -> lower=-5.4978 upper=0.15708 effort=1000.0 velocity=1.0

Commit message: use of stl in urdf

File: urdf/arm.urdf (robot description, URDF)
Before this commit: robot arm, 10 links, 9 joints
Links:
- added link gripper_center
- added link plate; visual mesh filename=package://arm_ros_conn/meshes/32985.stl
- link arm_base: geometry 
- link link1: geometry visual mesh filename=package://arm_ros_conn/meshes/link1.stl
- link link2: geometry visual mesh filename=package://arm_ros_conn/meshes/link2.stl
- link link3: geometry visual mesh filename=package://arm_ros_conn/meshes/link3.stl
- link link4: geometry visual mesh filename=package://arm_ros_conn/meshes/link4.stl
Joints:
- removed joint base_link_to_arm_base
- added joint base_link_to_plate: type fixed, parent base_link, child plate, origin xyz=0 0 0.00375
- added joint gripper_center_joint: type fixed, parent gripper_pole, child gripper_center, origin xyz=0.0 0.0 0.1 rpy=0 0 0
- added joint plate_to_arm_base: type fixed, parent plate, child arm_base, origin xyz=0 0.099 0
- joint arm_base_to_link1: origin xyz=0 0.099 0 -> (none)
- joint left_gripper_joint: origin xyz=0.02 0.01 0 rpy=0 0 0 -> xyz=0.0 0.01 0.02 rpy=0 -1.5708 0
- joint link_1_2_joint: axis 0 0 1 -> 0 1 0; limit lower=0.15045941827537324 upper=3.6110260386089577 effort=1000.0 velocity=1.0 -> lower=-2.0402 upper=1.4203 effort=1000.0 velocity=1.0; origin xyz=0.0 0.0 0.123 rpy=1.57075 0 0 -> xyz=0.0 0.0 0.123 rpy=0 0 0
- joint link_2_3_joint: axis 0 0 1 -> 0 1 0; limit lower=-3.141592653589793 upper=0.0 effort=1000.0 velocity=1.0 -> lower=-1.5708 upper=1.5708 effort=1000.0 velocity=1.0; origin xyz=0.240 0.0 0.0 rpy=0 0 0 -> xyz=0 0 0.240 rpy=0 0 0
- joint link_3_4_joint: axis 1 0 0 -> 0 0 1; origin xyz=0 0.135 0.0 rpy=1.57075 0 1.57075 -> xyz=0 0 0.135 rpy=0 0 0
- joint link_4_5_joint: origin xyz=0.06 0.0 0.0 rpy=0 0 0 -> xyz=0 0 0.06 rpy=0 0 0
- joint right_gripper_joint: origin xyz=0.02 -0.01 0 rpy=0 0 0 -> xyz=0.0 -0.01 0.02 rpy=0 -1.5708 0

Commit message: urdf joint angle to hw

File: urdf/arm.urdf (robot description, URDF)
Before this commit: robot arm, 12 links, 11 joints
Joints:
- removed joint arm_base_to_link1
- removed joint base_link_to_plate
- removed joint link_1_2_joint
- removed joint link_2_3_joint
- removed joint link_3_4_joint
- removed joint link_4_5_joint
- removed joint plate_to_arm_base
- added joint arm_base_joint: type fixed, parent plate, child arm_base, origin xyz=0 0.099 0
- added joint link1_joint: type revolute, parent arm_base, child link1, axis 0 0 -1, limit lower=0.0 upper=5.672320068981571 effort=1000.0 velocity=1.0
- added joint link2_joint: type revolute, parent link1, child link2, origin xyz=0.0 0.0 0.123 rpy=0 1.5708 0, axis 0 -1 0, limit lower=0.1505 upper=3.611 effort=1000.0 velocity=1.0
- added joint link3_joint: type revolute, parent link2, child link3, origin xyz=0 0 0.240 rpy=0 -1.5708 0, axis 0 1 0, limit lower=0 upper=3.1416 effort=1000.0 velocity=1.0
- added joint link4_joint: type revolute, parent link3, child link4, origin xyz=0 0 0.135 rpy=0 0 0, axis 0 0 -1, limit lower=-0.15708 upper=5.4978 effort=1000.0 velocity=1.0
- added joint link5_joint: type revolute, parent link4, child link5, origin xyz=0 0 0.06 rpy=0 0 0, axis 0 -1 0, limit lower=-1.5707963267948966 upper=1.5707963267948966 effort=1000.0 velocity=1.0
- added joint plate_joint: type fixed, parent base_link, child plate, origin xyz=0 0 0.00375

Commit message: urdf fixes

File: urdf/arm.urdf (robot description, URDF)
Before this commit: robot arm, 12 links, 11 joints
Joints:
- joint gripper_center_joint: origin xyz=0.0 0.0 0.1 rpy=0 0 0 -> xyz=0.08 0 0 rpy=0 0 0
- joint gripper_pole_joint: origin (none) -> xyz=0 0.02275 0 rpy=1.5708 0 1.5708
- joint left_gripper_joint: limit lower=0.0 upper=0.35 effort=1000.0 velocity=1.0 -> lower=0.0 upper=0.35 effort=1.0 velocity=1.0; origin xyz=0.0 0.01 0.02 rpy=0 -1.5708 0 -> xyz=0 0.015 0 rpy=0 0 0
- joint link1_joint: limit lower=0.0 upper=5.672320068981571 effort=1000.0 velocity=1.0 -> lower=0.0 upper=5.672320068981571 effort=1.0 velocity=1.0
- joint link2_joint: axis 0 -1 0 -> 0 0 1; limit lower=0.1505 upper=3.611 effort=1000.0 velocity=1.0 -> lower=0.1505 upper=3.611 effort=1.0 velocity=1.0; origin xyz=0.0 0.0 0.123 rpy=0 1.5708 0 -> xyz=0.0 0.0 0.123 rpy=1.5708 0 0
- joint link3_joint: axis 0 1 0 -> 0 0 -1; limit lower=0 upper=3.1416 effort=1000.0 velocity=1.0 -> lower=0 upper=3.1416 effort=1.0 velocity=1.0; origin xyz=0 0 0.240 rpy=0 -1.5708 0 -> xyz=0.240 0 0 rpy=0 0 0
- joint link4_joint: limit lower=-0.15708 upper=5.4978 effort=1000.0 velocity=1.0 -> lower=-0.15708 upper=5.4978 effort=1.0 velocity=1.0; origin xyz=0 0 0.135 rpy=0 0 0 -> xyz=0 0.135 0 rpy=-1.5708 0 0
- joint link5_joint: axis 0 -1 0 -> 0 0 1; limit lower=-1.5707963267948966 upper=1.5707963267948966 effort=1000.0 velocity=1.0 -> lower=-1.5707963267948966 upper=1.5707963267948966 effort=1.0 velocity=1.0; origin xyz=0 0 0.06 rpy=0 0 0 -> xyz=0 0 0.06 rpy=1.5708 0 0
- joint right_gripper_joint: axis 0 0 -1 -> 0 0 1; limit lower=0.0 upper=0.35 effort=1000.0 velocity=1.0 -> lower=0.0 upper=0.35 effort=1.0 velocity=1.0; origin xyz=0.0 -0.01 0.02 rpy=0 -1.5708 0 -> xyz=0 -0.015 0 rpy=3.1416 0 0

Commit message: urdf: updated velocities

File: urdf/arm.urdf (robot description, URDF)
Before this commit: robot arm, 12 links, 11 joints
Joints:
- joint left_gripper_joint: limit lower=0.0 upper=0.35 effort=1.0 velocity=1.0 -> lower=0.0 upper=0.35 effort=1.0 velocity=0.1
- joint link1_joint: limit lower=0.0 upper=5.672320068981571 effort=1.0 velocity=1.0 -> lower=0.0 upper=5.672320068981571 effort=1.0 velocity=0.1
- joint link2_joint: limit lower=0.1505 upper=3.611 effort=1.0 velocity=1.0 -> lower=0.1505 upper=3.611 effort=1.0 velocity=0.1
- joint link3_joint: limit lower=0 upper=3.1416 effort=1.0 velocity=1.0 -> lower=0 upper=3.1416 effort=1.0 velocity=0.1
- joint link4_joint: limit lower=-0.15708 upper=5.4978 effort=1.0 velocity=1.0 -> lower=-0.15708 upper=5.4978 effort=1.0 velocity=0.1
- joint link5_joint: limit lower=-1.5707963267948966 upper=1.5707963267948966 effort=1.0 velocity=1.0 -> lower=-1.5707963267948966 upper=1.5707963267948966 effort=1.0 velocity=0.1
- joint right_gripper_joint: limit lower=0.0 upper=0.35 effort=1.0 velocity=1.0 -> lower=0.0 upper=0.35 effort=1.0 velocity=0.1

Commit message: added pick_and_place.py

File: urdf/arm.urdf (robot description, URDF)
Before this commit: robot arm, 12 links, 11 joints
Joints:
- joint link1_joint: limit lower=0.0 upper=5.672320068981571 effort=1.0 velocity=0.1 -> lower=0.0 upper=5.672320068981571 effort=1.0 velocity=0.2
- joint link3_joint: limit lower=0 upper=3.1416 effort=1.0 velocity=0.1 -> lower=0 upper=3.1416 effort=1.0 velocity=0.2
- joint link4_joint: limit lower=-0.15708 upper=5.4978 effort=1.0 velocity=0.1 -> lower=-0.15708 upper=5.4978 effort=1.0 velocity=0.5
- joint link5_joint: limit lower=-1.5707963267948966 upper=1.5707963267948966 effort=1.0 velocity=0.1 -> lower=-1.5707963267948966 upper=1.5707963267948966 effort=1.0 velocity=1.0
